File: Hardware/6xUSB_PowMet.sch (KiCad schematic (older format))
At the start: 68 parts, among them IC1 ATMEGA32-M, P1 USB_A, P2 USB_A, P3 USB_A, P4 USB_A, P5 USB_A, P6 USB_A, P7 CONN_01X08, P8 CONN_01X03, P9 CONN_01X02, U1 LM1117MP-2.5, U2 LT6106, U3 LT6106, U4 LT6106, U5 LT6106, U6 LT6106, U7 LT6106

Commit message: Schematic updates
Parts:
- removed C18, C19, C20, C21, C22, C23: 10uF, Capacitors_SMD:C_0805_HandSoldering, symbol C_Small
- removed F1, F2, F3, F4, F5, F6: F_Small, Fuse_Holders_and_Fuses:Fuse_SMD1206_HandSoldering, symbol F_Small
- P1, P2, P3, P4, P5, P6: footprint USB-A_vertical1:USB_A_Vertical -> Connect:USB_A_Vertical
Connections:
- net labels removed: D1+, D1-, D2+, D2-, D3+, D3-, D4+, D4-
- wire segments 172 -> 155
- no-connect marks 24 -> 32
