File: USB_hub.sch (KiCad schematic (older format))
At the start: 43 parts, among them CON1 BARREL_JACK, P10 USB_B, Q1 IRFR5305PBF, U10 TPS5450-EP_DDA_8, U11 LTC4412, U8 AP1117E33, U9 FE1.1s, Y1 12Mhz

Commit message: Removed some files
Parts:
- Q1: footprint (none) -> TO_SOT_Packages_SMD1:TO-252-2Lead
Changed lines of the file:
@@
 $EndComp
 $Comp
-L Earth #PWR35
+L Earth #PWR031
 U 1 1 5717A71D
 P 4950 2750
-F 0 "#PWR35" H 4950 2500 50  0001 C CNN
+F 0 "#PWR031" H 4950 2500 50  0001 C CNN
 F 1 "Earth" H 4950 2600 50  0001 C CNN
 F 2 "" H 4950 2750 50  0000 C CNN
@@
 $EndComp
 $Comp
-L VCC #PWR34
+L VCC #PWR032
 U 1 1 5717B104
 P 4850 2400
-F 0 "#PWR34" H 4850 2250 50  0001 C CNN
+F 0 "#PWR032" H 4850 2250 50  0001 C CNN
 F 1 "VCC" H 4850 2550 50  0000 C CNN
 F 2 "" H 4850 2400 50  0000 C CNN
@@
 $EndComp
 $Comp
-L Earth #PWR36
+L Earth #PWR033
 U 1 1 5718DF93
 P 5850 4150
-F 0 "#PWR36" H 5850 3900 50  0001 C CNN
+F 0 "#PWR033" H 5850 3900 50  0001 C CNN
 F 1 "Earth" H 5850 4000 50  0001 C CNN
 F 2 "" H 5850 4150 50  0000 C CNN
@@
 $EndComp
 $Comp
-L VCC #PWR41
+L VCC #PWR034
 U 1 1 5718F538
 P 7500 1800
-F 0 "#PWR41" H 7500 1650 50  0001 C CNN
+F 0 "#PWR034" H 7500 1650 50  0001 C CNN
 F 1 "VCC" H 7500 1950 50  0000 C CNN
 F 2 "" H 7500 1800 50  0000 C CNN
@@
 $EndComp
 $Comp
-L Earth #PWR42
+L Earth #PWR035
 U 1 1 5718F80D
 P 7500 2500
-F 0 "#PWR42" H 7500 2250 50  0001 C CNN
+F 0 "#PWR035" H 7500 2250 50  0001 C CNN
 F 1 "Earth" H 7500 2350 50  0001 C CNN
 F 2 "" H 7500 2500 50  0000 C CNN
@@
 $EndComp
 $Comp
-L VCC #PWR44
+L VCC #PWR036
 U 1 1 57191069
 P 8250 3250
-F 0 "#PWR44" H 8250 3100 50  0001 C CNN
+F 0 "#PWR036" H 8250 3100 50  0001 C CNN
 F 1 "VCC" V 8250 3450 50  0000 C CNN
 F 2 "" H 8250 3250 50  0000 C CNN
@@
 $EndComp
 $Comp
-L Earth #PWR49
+L Earth #PWR037
 U 1 1 57197DDC
 P 9650 3200
-F 0 "#PWR49" H 9650 2950 50  0001 C CNN
+F 0 "#PWR037" H 9650 2950 50  0001 C CNN
 F 1 "Earth" H 9650 3050 50  0001 C CNN
 F 2 "" H 9650 3200 50  0000 C CNN
@@
 $EndComp
 $Comp
-L VCC #PWR45
+L VCC #PWR038
 U 1 1 5719A73E
 P 8450 3850
-F 0 "#PWR45" H 8450 3700 50  0001 C CNN
+F 0 "#PWR038" H 8450 3700 50  0001 C CNN
 F 1 "VCC" H 8450 4000 50  0000 C CNN
 F 2 "" H 8450 3850 50  0000 C CNN
@@
 $EndComp
 $Comp
-L Earth #PWR48
+L Earth #PWR039
 U 1 1 5719AF06
 P 9550 3650
-F 0 "#PWR48" H 9550 3400 50  0001 C CNN
+F 0 "#PWR039" H 9550 3400 50  0001 C CNN
 F 1 "Earth" H 9550 3500 50  0001 C CNN
 F 2 "" H 9550 3650 50  0000 C CNN
@@
 $EndComp
 $Comp
-L VCC #PWR47
+L VCC #PWR040
 U 1 1 5719B1E9
 P 9100 4200
-F 0 "#PWR47" H 9100 4050 50  0001 C CNN
+F 0 "#PWR040" H 9100 4050 50  0001 C CNN
 F 1 "VCC" H 9100 4350 50  0000 C CNN
 F 2 "" H 9100 4200 50  0000 C CNN
@@
 $EndComp
 $Comp
-L Earth #PWR50
+L Earth #PWR041
 U 1 1 571A242B
 P 10200 4500
-F 0 "#PWR50" H 10200 4250 50  0001 C CNN
+F 0 "#PWR041" H 10200 4250 50  0001 C CNN
 F 1 "Earth" H 10200 4350 50  0001 C CNN
 F 2 "" H 10200 4500 50  0000 C CNN
@@
 $EndComp
 $Comp
-L Earth #PWR51
+L Earth #PWR042
 U 1 1 571A25A5
 P 10800 4700
-F 0 "#PWR51" H 10800 4450 50  0001 C CNN
+F 0 "#PWR042" H 10800 4450 50  0001 C CNN
 F 1 "Earth" H 10800 4550 50  0001 C CNN
 F 2 "" H 10800 4700 50  0000 C CNN
@@
 $EndComp
 $Comp
-L Earth #PWR46
+L Earth #PWR043
 U 1 1 571A29D9
 P 8450 4550
-F 0 "#PWR46" H 8450 4300 50  0001 C CNN
+F 0 "#PWR043" H 8450 4300 50  0001 C CNN
 F 1 "Earth" H 8450 4400 50  0001 C CNN
 F 2 "" H 8450 4550 50  0000 C CNN
@@
 3V3
 $Comp
-L Earth #PWR40
+L Earth #PWR044
 U 1 1 571B4718
 P 6950 2050
-F 0 "#PWR40" H 6950 1800 50  0001 C CNN
+F 0 "#PWR044" H 6950 1800 50  0001 C CNN
 F 1 "Earth" H 6950 1900 50  0001 C CNN
 F 2 "" H 6950 2050 50  0000 C CNN
@@
 $EndComp
 $Comp
-L Earth #PWR39
+L Earth #PWR045
 U 1 1 571B493D
 P 6450 2050
-F 0 "#PWR39" H 6450 1800 50  0001 C CNN
+F 0 "#PWR045" H 6450 1800 50  0001 C CNN
 F 1 "Earth" H 6450 1900 50  0001 C CNN
 F 2 "" H 6450 2050 50  0000 C CNN
@@
 $EndComp
 $Comp
-L Earth #PWR38
+L Earth #PWR046
 U 1 1 571B4AB5
 P 6000 1350
-F 0 "#PWR38" H 6000 1100 50  0001 C CNN
+F 0 "#PWR046" H 6000 1100 50  0001 C CNN
 F 1 "Earth" H 6000 1200 50  0001 C CNN
 F 2 "" H 6000 1350 50  0000 C CNN
@@
 $EndComp
 $Comp
-L VCC #PWR37
+L VCC #PWR047
 U 1 1 571B4C02
 P 5950 1750
-F 0 "#PWR37" H 5950 1600 50  0001 C CNN
+F 0 "#PWR047" H 5950 1600 50  0001 C CNN
 F 1 "VCC" H 5950 1900 50  0000 C CNN
 F 2 "" H 5950 1750 50  0000 C CNN
@@
 Connection ~ 7100 5200
 $Comp
-L Earth #PWR43
+L Earth #PWR048
 U 1 1 5730ABC1
 P 7550 5900
-F 0 "#PWR43" H 7550 5650 50  0001 C CNN
+F 0 "#PWR048" H 7550 5650 50  0001 C CNN
 F 1 "Earth" H 7550 5750 50  0001 C CNN
 F 2 "" H 7550 5900 50  0000 C CNN
@@
 VCC
 $Comp
-L Earth #PWR32
+L Earth #PWR049
 U 1 1 5730CFDB
 P 2500 5600
-F 0 "#PWR32" H 2500 5350 50  0001 C CNN
+F 0 "#PWR049" H 2500 5350 50  0001 C CNN
 F 1 "Earth" H 2500 5450 50  0001 C CNN
 F 2 "" H 2500 5600 50  0000 C CNN
@@
 F 0 "Q1" H 4000 1200 50  0000 R CNN
 F 1 "IRFR5305PBF" H 4050 1100 50  0000 R CNN
-F 2 "" H 3900 1250 50  0000 C CNN
+F 2 "TO_SOT_Packages_SMD1:TO-252-2Lead" H 3900 1250 50  0001 C CNN
 F 3 "" H 3700 1150 50  0000 C CNN
 	1    3700 1150
@@
 	2250 1700 2250 1850
 $Comp
-L Earth #PWR31
+L Earth #PWR050
 U 1 1 5734467A
 P 2250 1850
-F 0 "#PWR31" H 2250 1600 50  0001 C CNN
+F 0 "#PWR050" H 2250 1600 50  0001 C CNN
 F 1 "Earth" H 2250 1700 50  0001 C CNN
 F 2 "" H 2250 1850 50  0000 C CNN
@@
 $EndComp
 $Comp
-L Earth #PWR33
+L Earth #PWR051
 U 1 1 57344A03
 P 4300 1450
-F 0 "#PWR33" H 4300 1200 50  0001 C CNN
+F 0 "#PWR051" H 4300 1200 50  0001 C CNN
 F 1 "Earth" H 4300 1300 50  0001 C CNN
 F 2 "" H 4300 1450 50  0000 C CNN
