File: Hardware/PCB/6xUSB_PowMet.sch (KiCad schematic (older format))
At the start: 68 parts, among them IC1 ATMEGA32-M, P1 USB_A, P2 USB_A, P3 USB_A, P4 USB_A, P5 USB_A, P6 USB_A, P7 CONN_01X06, P8 CONN_01X03, P9 CONN_01X03, U1 LM1117MP-2.5, U2 LT6106, U3 LT6106, U4 LT6106, U5 LT6106, U6 LT6106, U7 LT6106

Commit message: Upd_sch
Updated schematic and PCB
Parts:
- R5: value 14K -> 15K
Changed lines of the file:
@@
 P 5900 1800
 F 0 "R5" V 5980 1800 50  0000 C CNN
-F 1 "14K" V 5900 1800 50  0000 C CNN
+F 1 "15K" V 5900 1800 50  0000 C CNN
 F 2 "Resistors_SMD:R_0805" V 5830 1800 50  0001 C CNN
 F 3 "" H 5900 1800 50  0000 C CNN

Commit message: Upd
Schematic updates and PCB
Parts:
- removed C5: 100n, Capacitors_SMD:C_0805, symbol C
- removed C6: 10uF, Capacitors_Tantalum_SMD:TantalC_SizeC_EIA-6032_HandSoldering, symbol CP1_Small
- removed U1: LM1117MP-2.5, TO_SOT_Packages_SMD:SOT-223, symbol LM1117MP-2.5
- added C5: 100n, Capacitors_SMD:C_0805, symbol C_Small
- added C6: 10uF, Capacitors_SMD:C_0805, symbol C_Small
- added U1: LM1117MP-2.5, TO_SOT_Packages_SMD:SOT-223, symbol LM1117MP-v.v
- P7: footprint Connect:Wafer_Vertical20x5.8x7RM2.5-7 -> Connect:Wafer_Vertical17.5x5.8x7RM2.5-6
Connections:
- net +2.5V: now also C6.1, U1.2 (OUT)
- net GND: now also C5.2, C6.2, U1.1
- net VCC: now also C5.1, U1.3 (IN)
- net PC6_25: now reaches IC1.25 ((TOSC1)PC6)
- net PC7_26: now reaches IC1.26 ((TOSC2)PC7)
- no-connect marks 24 -> 22

Commit message: updates
Parts:
- removed C1, C10, C11, C15, C16, C17, C8, C9: 100n, Capacitors_SMD:C_0805, symbol C
- removed C12, C13, C14, C2, C3, C4, C7: 1n, Capacitors_SMD:C_0805, symbol C
- removed C18, C19, C20, C21, C22, C23: 10uF, Capacitors_SMD:C_0805_HandSoldering, symbol C_Small
- removed C5: 100n, Capacitors_SMD:C_0805, symbol C_Small
- removed C6: 10uF, Capacitors_SMD:C_0805, symbol C_Small
- removed F2, F3, F4, F5, F6: F_Small, Fuse_Holders_and_Fuses:Fuse_SMD1206_HandSoldering, symbol F_Small
- removed IC1: ATMEGA32-M, Housings_QFP:TQFP-44_10x10mm_Pitch0.8mm, symbol ATMEGA32-M
- removed L1: 10uH, Inductors:Inductor_1212, symbol L
- removed P2, P3, P4, P5, P6: USB_A, USB-A_vertical1:USB_A_Vertical, symbol USB_A
- removed P7: CONN_01X06, Connect:Wafer_Vertical17.5x5.8x7RM2.5-6, symbol CONN_01X06
- removed P8, P9: CONN_01X03, Connect:Wafer_Vertical10x5.8x7RM2.5-3, symbol CONN_01X03
- removed R1, R10, R16, R17, R19, R9: 100R, Resistors_SMD:R_0805, symbol R
- removed R11, R12, R18, R2, R20, R21: 0.01R, Resistors_SMD:R_0805, symbol R
- removed R13, R14, R15, R3, R4, R7, R8: 10K, Resistors_SMD:R_0805, symbol R
- removed R6: 10k, Resistors_SMD:R_0805, symbol R
- removed U1: LM1117MP-2.5, TO_SOT_Packages_SMD:SOT-223, symbol LM1117MP-v.v
- removed U2, U3, U4, U5, U6, U7: LT6106, TO_SOT_Packages_SMD:SOT-23-5, symbol LT6106
- added C1: 10n, Capacitors_SMD:C_0805, symbol Device:C_Small
- added C10, C3, C4, C6, C7, C8, C9: 100n, Capacitors_SMD:C_0805, symbol Device:C_Small
- added C11: 1nF, Capacitors_SMD:C_0805, symbol Device:C_Small
- added C18, C19, C36, C44: 10uF, Capacitors_SMD:C_0805, symbol Device:C_Small
- added C2: 0.33uF, Capacitors_SMD:C_0805, symbol Device:C_Small
- added C25, C32: 22pF, Capacitors_SMD:C_0603, symbol Device:C_Small
- added C46: 22uF, Capacitors_Tantalum_SMD:CP_Tantalum_Case-R_EIA-2012-12_Reflow, symbol Device:CP1_Small
- added C47, C49: 1uF, Capacitors_SMD:C_0805, symbol Device:C
- added C5: 33nF, Capacitors_SMD:C_0805, symbol Device:C_Small
- added D3: CD1206-S01575, Diodes_SMD:D_1206, symbol Device:D
- added F2, F4, F5: F_Small, Fuse_Holders_and_Fuses:Fuse_SMD1206_Reflow, symbol 6xUSB_PowMet-rescue:F_Small
- added F8: MSMF050-2, Resistors_SMD:R_1812, symbol Device:Fuse_Small
- added J1: MICROUSB, kicad-libs-master:USB-MICRO-B-FCI-10118193, symbol 6xUSB_PowMet-rescue:MICROUSB-microusb
- added J2: CONN_01X04, Connectors_JST:JST_EH_B04B-EH-A_04x2.50mm_Straight, symbol 6xUSB_PowMet-rescue:CONN_01X04
- added J3: CONN_01X11, Connectors_JST:JST_EH_B11B-EH-A_11x2.50mm_Straight, symbol 6xUSB_PowMet-rescue:CONN_01X11
- added L1: MH2029-300Y, Inductors_SMD:L_0805, symbol Device:Ferrite_Bead
- added L11, L12, L8, L9: WE-CBF, Inductors_SMD:L_0603, symbol Device:L_Small
- added P2, P4, P5: USB_A, USB_A_Vertical:USB_A_Vertical, symbol 6xUSB_PowMet-rescue:USB_A-RESCUE-6xUSB_PowMet
- added Q10, Q5, Q7, Q9: IRLML6401, TO_SOT_Packages_SMD:SOT-23, symbol 6xUSB_PowMet-rescue:P-CHAN-MOSFET_SOT
- added R1: R_PHOTO, symbol Device:R_PHOTO
- added R10, R11, R12, R15, R4, R6, R8, R9: 10K, Resistors_SMD:R_0805, symbol Device:R_Small
- added R13, R16, R17, R2: 0.0025R, Resistors_SMD:R_1206, symbol Device:R
- added R14: 100R, Resistors_SMD:R_0805, symbol Device:R_Small
- added R3: 100K, Resistors_SMD:R_0805, symbol Device:R_Small
- added R32, R7: 22R, Resistors_SMD:R_0805, symbol Device:R
- added RV1, RV2: CG0603MLC-05E, Inductors_SMD:L_0603, symbol 6xUSB_PowMet-rescue:VDR
- added SW2: Reset, Buttons_Switches_SMD:SW_SPST_B3U-3000P, symbol 6xUSB_PowMet-rescue:SW_PUSH
- added TP1: TEST, Measurement_Points:Measurement_Point_Round-SMD-Pad_Small, symbol 6xUSB_PowMet-rescue:TEST
- added U12: 5v to 3.3v LDO, TO_SOT_Packages_SMD:SOT-223-3Lead_TabPin2, symbol regul:L7805
- added U3: ATMEGA32U4-AU, Housings_QFP:LQFP-44_10x10mm_Pitch0.8mm, symbol atmel:ATMEGA32U4-AU
- added U5: MAX34406FETG+, agg:QFN-40-EP-LTC-UJ, symbol 6xUSB_PowMet-rescue:MAX34406FETG+
- added U8: LM4040N-4.1, TO_SOT_Packages_SMD:SOT-23, symbol 6xUSB_PowMet-rescue:LM4040AvvDBZ
- added Y2: 16.000 Mhz, Crystals:Crystal_SMD_5032-4pin_5.0x3.2mm, symbol Device:Crystal_GND24_Small
- F1: footprint Fuse_Holders_and_Fuses:Fuse_SMD1206_HandSoldering -> Fuse_Holders_and_Fuses:Fuse_SMD1206_Reflow; symbol F_Small -> 6xUSB_PowMet-rescue:F_Small; Description (none) -> Fuse Chip Slow Blow Acting 3.5A 63V SMD Solder Pad 1206 Cer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; Manufacturer (none) -> BEL Group; Part Number (none) -> C1S 3.5
- P1: footprint USB-A_vertical1:USB_A_Vertical -> USB_A_Vertical:USB_A_Vertical; symbol USB_A -> 6xUSB_PowMet-rescue:USB_A-RESCUE-6xUSB_PowMet; Description (none) -> USB Connectors WR-COM USB Type A THT UpRight Short; Manufacturer (none) -> Wurth Electronics; Part Number (none) -> 614004184726
- R5: symbol R -> Device:R; Description (none) -> Thick Film Resistors - SMD 15K OHM 5%; Manufacturer (none) -> Yageo; Part Number (none) -> RC0805JR-0715KL; Tolerance (none) -> 5%
Connections:
- net labels added: +3V3, +3v3, +4.096V, ADC10, ADC9, D+, D-, ENA, MC_ST, PB0_40, SHTDN, USB_1, USB_2, USB_3, USB_4, USB_P, VBUS, WE-TVS_824001
- net labels removed: +2.5V, PC6_25, PC7_26
- wire segments 174 -> 258
- no-connect marks 22 -> 3
Other:
- note added: "3v3 power for ESP"
- note added: "AREF 4.1V"
- note added: "USB ESD EMI protection"
- note added: "uC Reset"
- note added: "uC USB flashing"
- moved on the sheet: F1, P1, R5
