File: Hardware/PCB/USB_hub.sch (KiCad schematic (older format))
At the start: 43 parts, among them CON1 BARREL_JACK, P10 USB_B, Q1 IRFR5305PBF, U10 TPS5450-EP_DDA_8, U11 LTC4412, U8 AP1117E33, U9 FE1.1s, Y1 12Mhz

Commit message: Updated pcb
Updated schematic and solved some pcb mistakes
Parts:
- L2: value INDUCTOR_SMALL -> 10uH; footprint (none) -> Inductors_NEOSID:Neosid_Inductor_SM-NE56_SMD2220
Changed lines of the file:
@@
 EESchema Schematic File Version 2
-LIBS:TPS5450-EP_DDA_8
 LIBS:power
 LIBS:device
@@
 LIBS:contrib
 LIBS:valves
-LIBS:tm-kicad-lib
-LIBS:TPS5450_DDA_8
-LIBS:tom_kicad
 LIBS:6xUSB_PowMet-cache
 EELAYER 25 0
@@
 P 8050 5200
 F 0 "L2" H 8050 5300 50  0000 C CNN
-F 1 "INDUCTOR_SMALL" H 8050 5150 50  0000 C CNN
-F 2 "" H 8050 5200 50  0000 C CNN
+F 1 "10uH" H 8050 5150 50  0000 C CNN
+F 2 "Inductors_NEOSID:Neosid_Inductor_SM-NE56_SMD2220" H 8050 5200 50  0001 C CNN
 F 3 "" H 8050 5200 50  0000 C CNN
 	1    8050 5200

Commit message: Upd_sch
Updated schematic and PCB
Parts:
- Y1: footprint Crystals:Crystal_HC49-SD_SMD -> Crystals:Crystal_SMD_5032_4Pads; symbol Crystal_Small -> CRYSTAL_SMD
Connections:
- wire segments 139 -> 142
Changed lines of the file:
@@
 $EndComp
 $Comp
-L Crystal_Small Y1
+L CRYSTAL_SMD Y1
 U 1 1 5717A09F
-P 5550 3200
-F 0 "Y1" H 5550 3300 50  0000 C CNN
-F 1 "12Mhz" H 5550 3100 50  0000 C CNN
-F 2 "Crystals:Crystal_HC49-SD_SMD" H 5550 3200 50  0001 C CNN
-F 3 "" H 5550 3200 50  0000 C CNN
-	1    5550 3200
+P 5450 3100
+F 0 "Y1" H 5450 3200 50  0000 C CNN
+F 1 "12Mhz" H 5450 3000 50  0000 C CNN
+F 2 "Crystals:Crystal_SMD_5032_4Pads" H 5450 3100 50  0001 C CNN
+F 3 "" H 5450 3100 50  0000 C CNN
+	1    5450 3100
 	0    1    1    0
 $EndComp
@@
 	5750 3000 5750 3150
 Wire Wire Line
-	5550 3300 5750 3300
+	5450 3300 5750 3300
 Wire Wire Line
 	5750 3300 5750 3250
@@
 Wire Wire Line
 	3900 2750 4950 2750
-Wire Wire Line
-	5550 3100 5550 3050
 Wire Wire Line
 	5550 3050 5750 3050
@@
 Text GLabel 10100 4200 1    60   Input ~ 0
 VREG
+Wire Wire Line
+	5550 3050 5550 2900
+Wire Wire Line
+	5550 2900 5450 2900
+Wire Wire Line
+	5350 3100 5300 3100
+Wire Wire Line
+	5300 3100 5300 3250
+$Comp
+L Earth #PWR052
+U 1 1 5746C36B
+P 5300 3250
+F 0 "#PWR052" H 5300 3000 50  0001 C CNN
+F 1 "Earth" H 5300 3100 50  0001 C CNN
+F 2 "" H 5300 3250 50  0000 C CNN
+F 3 "" H 5300 3250 50  0000 C CNN
+	1    5300 3250
+	1    0    0    -1
+$EndComp
 $EndSCHEMATC

Commit message: Updates schematic
Updated schematic and added datasheets
Parts:
- removed C32, C33: 47uF, Capacitors_SMD:C_1206_HandSoldering, symbol C_Small
- removed C34: 10n, Capacitors_SMD:C_0805_HandSoldering, symbol C_Small
- removed C35: 180uF, Capacitors_SMD:c_elec_8x10.5, symbol CP1_Small
- removed CON1: BARREL_JACK, Connect:JACK_ALIM, symbol BARREL_JACK
- removed D8: D_Schottky, Diodes_SMD:SMC_Handsoldering, symbol D_Schottky
- removed L2: 10uH, Inductors_NEOSID:Neosid_Inductor_SM-NE56_SMD2220, symbol INDUCTOR_SMALL
- removed R31: 10K, Resistors_SMD:R_0805_HandSoldering, symbol R_Small
- removed R32: 3.24K, Resistors_SMD:R_0805_HandSoldering, symbol R_Small
- removed U10: TPS5450-EP_DDA_8, TPS5450-EP_DDA_8:DDA8_3X2P49, symbol TPS5450-EP_DDA_8
- added C37: 22uF, Capacitors_SMD:C_1206, symbol C_Small
- added C38: 100nF, Capacitors_SMD:C_0805, symbol C_Small
- added C39: 15nF, Capacitors_SMD:C_0805, symbol C_Small
- added C40: 470nF, Capacitors_SMD:C_0805, symbol C_Small
- added C41: 1uF, Capacitors_SMD:C_0805, symbol C_Small
- added C42: 470pF, Capacitors_SMD:C_0805, symbol C_Small
- added C43: 220uF, Capacitors_SMD:c_elec_6.3x5.3, symbol CP1_Small
- added CON2: BARREL_JACK, Connect:JACK_ALIM, symbol BARREL_JACK
- added D10: SKL14, Diodes_SMD:SOD-123, symbol D_Schottky
- added D11: SK2030YD2, Diodes_SMD:DD-PAK_TO263_DualDiode, symbol SCHDPAK
- added D9, D? (x2): Power, LEDs:LED-5MM, symbol Led_Small
- added L3: 2.2uH, Inductors:SELF-WE-PD-XXL, symbol INDUCTOR_SMALL
- added Q2: CSD16342Q5A, MICRO8, symbol IRF7607PBF
- added Q3: CSD17577Q5A, MICRO8, symbol IRF7607PBF
- added R34: 100K, Resistors_SMD:R_0805, symbol R_Small
- added R35: 1K07, Resistors_SMD:R_0805, symbol R_Small
- added R36: 73K2, Capacitors_SMD:C_0805, symbol R_Small
- added R37: 10K, Capacitors_SMD:C_0805, symbol R_Small
- added R38, R? (x2): 330, Resistors_SMD:R_0805_HandSoldering, symbol R_Small
- added U12: 74HC08, Housings_SOIC:SOIC-14_3.9x8.7mm_Pitch1.27mm, symbol 7408
- added U13: LM3150, IPC7351-Nominal:SOP65P640X120-15, symbol LM3150
- F7: value F_Small -> 500mA
Connections:
- net labels added: USB_P
- wire segments 142 -> 180
- no-connect marks 5 -> 3
Other:
- moved on the sheet: D1, F7, P10, R22

Commit message: Upd
Schematic updates and PCB
Parts:
- removed U12: 74HC08, Housings_SOIC:SOIC-14_3.9x8.7mm_Pitch1.27mm, symbol 7408
- C24: value 4.7uF -> 10uF
- C25: value 4.7uF -> 22uF
- D2, D3, D4, D5, D6: footprint LEDs:LED-5MM -> LEDs:LED_0805
- D7: footprint Diodes_SMD:SMC_Standard -> Diodes_SMD:MiniMELF_Standard
- P10: footprint (none) -> Connect:USB_B
- Q2, Q3: footprint MICRO8 -> Personal:AB2_SON5x6_FET
- U13: footprint IPC7351-Nominal:SOP65P640X120-15 -> Housings_SSOP:SSOP-14_5.3x6.2mm_Pitch0.65mm
- U8: footprint TO_SOT_Packages_SMD:SOT89-3_Housing_Handsoldering -> TO_SOT_Packages_SMD:SOT-223
- U9: footprint Housings_SSOP:SSOP-28_5.3x10.2mm_Pitch0.65mm -> Housings_SSOP:TSSOP-28_4.4x9.7mm_Pitch0.65mm
- gave numbers to parts that had none: 4
Connections:
- net PC6_25: now reaches R32.1
- net PC7_26: now reaches R31.1
- net 3V3 renamed +3.3V

Commit message: updates
Parts:
- removed C24, C30, C31: 10uF, Capacitors_SMD:C_0805_HandSoldering, symbol C_Small
- removed C25: 22uF, Capacitors_SMD:C_0805_HandSoldering, symbol C_Small
- removed C27: 10pF, Capacitors_SMD:C_0805_HandSoldering, symbol C_Small
- removed C29: 10nF, Capacitors_SMD:C_0805_HandSoldering, symbol C_Small
- removed C36: 100nF, Capacitors_SMD:C_0805_HandSoldering, symbol C_Small
- removed D1, D12, D8: Power, LEDs:LED-5MM, symbol Led_Small
- removed D3, D4, D5: Led_Small, LEDs:LED_0805, symbol Led_Small
- removed D7: 5.1V, Diodes_SMD:MiniMELF_Standard, symbol D_Schottky_Small
- removed F7: 500mA, Fuse_Holders_and_Fuses:Fuse_SMD1206_HandSoldering, symbol F_Small
- removed R22, R24, R25, R31, R32, R38: 330, Resistors_SMD:R_0805_HandSoldering, symbol R_Small
- removed R26, R28, R30: 10K, Resistors_SMD:R_0805_HandSoldering, symbol R_Small
- removed U8: AP1117E33, TO_SOT_Packages_SMD:SOT-223, symbol AP1117E33
- added C24, C30, C33: 0.1uF, Capacitors_SMD:C_0603, symbol Device:C_Small
- added C29: 10nF, Capacitors_SMD:C_0805, symbol Device:C_Small
- added C31, C51: 47uF, Capacitors_SMD:C_1206, symbol Device:C_Small
- added C48: 100n, Capacitors_SMD:C_0805, symbol Device:C_Small
- added C52: 18pF, Capacitors_SMD:C_0805, symbol Device:C_Small
- added D1: USB Power, LEDs:LED_D3.0mm_Horizontal_O6.35mm_Z6.0mm, symbol 6xUSB_PowMet-rescue:Led_Small
- added D2: MC Status, LEDs:LED_0603, symbol 6xUSB_PowMet-rescue:Led_Small
- added F7: MSMF050-2, Resistors_SMD:R_1812, symbol Device:Fuse_Small
- added L10, L2, L5, L6, L7: WE-CNSW, Inductors_SMD:L_CommonMode_Wuerth_WE-CNSW, symbol 6xUSB_PowMet-rescue:L_Core_double_Iron_Small
- added L4: Bead/100MHZ/470ohm/2A, Resistors_SMD:R_0805_HandSoldering, symbol 6xUSB_PowMet-rescue:INDUCTOR_SMALL
- added LED1, LED2, LED3: Led_Small, Inductors_SMD:L_1806, symbol 6xUSB_PowMet-rescue:Led_Small
- added R26, R42: 10K, Resistors_SMD:R_0805, symbol Device:R_Small
- added R28, R38, R45: 100K, Resistors_SMD:R_0805, symbol Device:R_Small
- added R31: 330, Resistors_SMD:R_0805, symbol Device:R_Small
- added R46: 470R, Resistors_SMD:R_0805, symbol Device:R_Small
- added R47: 100R, Resistors_SMD:R_0805, symbol Device:R_Small
- added R48, R49: 150R, Resistors_SMD:R_0805, symbol Device:R_Small
- added U1: 24LC02, Housings_SOIC:SOIC-8_3.9x4.9mm_Pitch1.27mm, symbol memory:24LC02
- C26: value 10pF -> 18pF; footprint Capacitors_SMD:C_0805_HandSoldering -> Capacitors_SMD:C_0805; symbol C_Small -> Device:C_Small; Description (none) -> Cap Ceramic 18pF 50V C0G 5% Pad SMD 0805 125°C T/R; Manufacturer (none) -> Samsung Electro-Mechanics; Material (none) -> Ceramic; Part Number (none) -> CL21C180JBANNNC; Tolerance (none) -> 5%; Voltage (none) -> 50V
- C28: footprint Capacitors_SMD:C_0805_HandSoldering -> Capacitors_SMD:C_0805; symbol C_Small -> Device:C_Small; Description (none) -> Cap Ceramic 10uF 16V X5R 10% Pad SMD 0805 85°C T/R; Manufacturer (none) -> Taiyo Yuden; Material (none) -> Ceramix X5R; Part Number (none) -> EMK212ABJ106KG-T; Tolerance (none) -> 10%; Voltage (none) -> 16V
- C37: value 22uF -> 47uF; symbol C_Small -> Device:C_Small; Description (none) -> Cap Ceramic 47uF 25V X5R 20% Pad SMD 1206 85°C T/R; Manufacturer (none) -> TDK; Material (none) -> Ceramic X5R; Part Number (none) -> C3216X5R1E476M160AC; Tolerance (none) -> 10%; Voltage (none) -> 25V
- C38: value 100nF -> 100n; symbol C_Small -> Device:C_Small; Description (none) -> Cap Ceramic 0.1uF 25V X7R 10% Pad SMD 0805 125°C T/R; Manufacturer (none) -> AVX; Material (none) -> Ceramic X7R; Part Number (none) -> 08053C104KAT2A; Tolerance (none) -> 10%; Voltage (none) -> 25V
- C39: symbol C_Small -> Device:C_Small; Description (none) -> Cap Ceramic 0.015uF 50V X7R 10% Pad SMD 0805 125°C T/R; Manufacturer (none) -> Yageo; Material (none) -> Ceramic X7R; Part Number (none) -> CC0805KRX7R9BB153; Tolerance (none) -> 10%; Voltage (none) -> 50V
- C40: symbol C_Small -> Device:C_Small; Description (none) -> Cap Ceramic 0.47uF 16V X7R 10% Pad SMD 0805 125°C T/R; Manufacturer (none) -> Taiyo Yuden; Material (none) -> Ceramic X7R; Part Number (none) -> EMK212B7474KD-T; Tolerance (none) -> 10%; Voltage (none) -> 16V
- C41: symbol C_Small -> Device:C_Small; Description (none) -> Cap Ceramic 1uF 16V X7R 10% Pad SMD 0805 125°C T/R; Manufacturer (none) -> Taiyo Yuden; Material (none) -> Ceramic X7R; Part Number (none) -> EMK212B7105KG-T; Tolerance (none) -> 10%; Voltage (none) -> 16V
- C42: value 470pF -> 1nF; symbol C_Small -> Device:C_Small; Description (none) -> Cap Ceramic 0.001uF 50V X7R 10% Pad SMD 0805 125°C T/R; Manufacturer (none) -> KEMET Corporation; Material (none) -> Ceramic X7R; Part Number (none) -> C0805C102K5RACTU; Tolerance (none) -> 10%; Voltage (none) -> 50V
- C43: value 220uF -> 330uF; footprint Capacitors_SMD:c_elec_6.3x5.3 -> Capacitors_SMD:CP_Elec_6.3x5.8; symbol CP1_Small -> Device:CP1_Small; Description (none) -> Cap Aluminum Polymer 330uF 6.3VDC 20% (6.3 X 5.9mm) SMD 0.0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; Manufacturer (none) -> Panasonic; Material (none) -> Aluminium; Part Number (none) -> 6SVPC330M; Tolerance (none) -> 20%; Voltage (none) -> 6V3
- CON2: symbol BARREL_JACK -> 6xUSB_PowMet-rescue:BARREL_JACK-connectors; Description (none) -> Conn Power F 2 POS Solder RA Thru-Hole 2 Terminal 1 Port; Manufacturer (none) -> CUI Inc; Part Number (none) -> PJ-082BH
- D10: symbol D_Schottky -> Device:D_Schottky; Description (none) -> Diode Schottky 20V 1A 2-Pin SOD-123FL T/R; Manufacturer (none) -> Micro Commercial Components; Part Number (none) -> SM5817PL-TP; Поле4 Schottky diode 1 A 40 V -> (none)
- D11: value SK2030YD2 -> SK152-TP; footprint Diodes_SMD:DD-PAK_TO263_DualDiode -> agg:DO-214AB-SMC; symbol SCHDPAK -> 6xUSB_PowMet-rescue:SCHDPAK; Description (none) -> Diode Schottky 20V 15A 2-Pin HSMC T/R; Manufacturer (none) -> Micro Commercial Components; Part Number (none) -> SK152-TP
- D6: value Led_Small -> Led_Small_3mm; footprint LEDs:LED_0805 -> LEDs:LED_D3.0mm_Horizontal_O6.35mm_Z6.0mm; symbol Led_Small -> 6xUSB_PowMet-rescue:Led_Small; Description (none) -> Standard LEDs - Red Through Hole Red Diffused; Manufacturer (none) -> Lite-On; Part Number (none) -> MCL034MD
- D9: value Power -> Power DC; footprint LEDs:LED-5MM -> LEDs:LED_D3.0mm_Horizontal_O6.35mm_Z6.0mm; symbol Led_Small -> 6xUSB_PowMet-rescue:Led_Small; Description (none) -> LED Uni-Color Red Orange 630nm 2-Pin T-1; Manufacturer (none) -> Lite-On Technology; Part Number (none) -> LTL-4291N
- L3: value 2.2uH -> 4.7uH 5.2mOhm; footprint Inductors:SELF-WE-PD-XXL -> (none); symbol INDUCTOR_SMALL -> 6xUSB_PowMet-rescue:INDUCTOR_SMALL; Manufacturer (none) -> Coilcraft; Part Number (none) -> XAL1010-472MEB
- LED4: renamed from D2; footprint LEDs:LED_0805 -> Inductors_SMD:L_1806; symbol Led_Small -> 6xUSB_PowMet-rescue:Led_Small; Manufacturer (none) -> Kingbright; Part Number (none) -> APA3010CGCK-GX
- P10: symbol USB_B -> 6xUSB_PowMet-rescue:USB_B-RESCUE-6xUSB_PowMet; Description (none) -> USB Connectors USB 2.0 type B jack 4 pin Horizontal TH; Manufacturer (none) -> CUI; Part Number (none) -> UJ2-BH-1-TH
- Q1: symbol Q_PMOS_GDS -> Device:Q_PMOS_GDS; Description (none) -> Trans MOSFET P-CH Si 55V 31A 3-Pin(2+Tab) DPAK Tube; Manufacturer (none) -> Infineon Technologies; Part Number (none) -> IRFR5305TRLPBF
- Q2: value CSD16342Q5A -> CSD16321Q5; symbol IRF7607PBF -> transistors:IRF7607PBF; Description (none) -> Trans MOSFET N-CH 25V 31A 8-Pin VSON-CLIP EP T/R; Manufacturer (none) -> Texas Instruments; Part Number (none) -> CSD16321Q5
- Q3: value CSD17577Q5A -> CSD18509Q5B; symbol IRF7607PBF -> transistors:IRF7607PBF; Description (none) -> Trans MOSFET N-CH Si 40V 100A 8-Pin VSON-CLIP EP T/R; Manufacturer (none) -> Texas Instruments; Part Number (none) -> CSD18509Q5B
- R23: value 330 -> 100R; footprint Resistors_SMD:R_0805_HandSoldering -> Resistors_SMD:R_0805; symbol R_Small -> Device:R_Small; Description (none) -> Thick Film Resistors 100 OHM 5%; Manufacturer (none) -> Yageo; Part Number (none) -> RC0805JR-07100RL; Tolerance (none) -> 5%
- R27: footprint Resistors_SMD:R_0805_HandSoldering -> Resistors_SMD:R_0805; symbol R_Small -> Device:R_Small; Description (none) -> Res Thick Film 0805 10K Ohm 5% 0.125W(1/8W) ±100ppm/°C Epox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; Manufacturer (none) -> Yageo; Part Number (none) -> RC0805JR-0710KL
- R29: footprint Resistors_SMD:R_0805_HandSoldering -> Resistors_SMD:R_0805; symbol R_Small -> Device:R_Small; Manufacturer (none) -> MULTICOMP; Part Number (none) -> MCWR08X2701FTL; Tolerance (none) -> 1%; Voltage (none) -> 150V
- R33: footprint Resistors_SMD:R_0805_HandSoldering -> Resistors_SMD:R_0805; symbol R_Small -> Device:R_Small; Description (none) -> Thick Film Resistors - SMD 470K OHM 5%; Manufacturer (none) -> Yageo; Part Number (none) -> RC0805JR-07470KL; Tolerance (none) -> 5%
- R34: value 100K -> 237K; symbol R_Small -> Device:R_Small; Description (none) -> Res Thick Film 0805 237K Ohm 1% 0.125W(1/8W) ±100ppm/°C Pad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; Manufacturer (none) -> Panasonic; Part Number (none) -> ERJ-6ENF2373V; Tolerance (none) -> 1%
- R35: symbol R_Small -> Device:R_Small; Description (none) -> Res Thick Film 0805 464 Ohm 1% 0.125W(1/8W) ±100ppm/°C Pad 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; Manufacturer (none) -> Vishay; Part Number (none) -> CRCW0805464RFKEA; Tolerance (none) -> 1%
- R36: footprint Capacitors_SMD:C_0805 -> Resistors_SMD:R_0805; symbol R_Small -> Device:R_Small; Description (none) -> Res Thick Film 0805 73.2K Ohm 1% 0.125W(1/8W) ±100ppm/°C Pa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; Manufacturer (none) -> Panasonic; Part Number (none) -> ERJ-6ENF7322V; Tolerance (none) -> 1%
- R37: footprint Capacitors_SMD:C_0805 -> Resistors_SMD:R_0805; symbol R_Small -> Device:R_Small; Description (none) -> Res Thick Film 0805 10K Ohm 1% 0.125W(1/8W) ±100ppm/°C Pad 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; Manufacturer (none) -> Panasonic; Part Number (none) -> ERJ-6ENF1002V; Tolerance (none) -> 1%
- U11: footprint tom_kicad_lib:SOT-6 -> TO_SOT_Packages_SMD:SOT-23-6; symbol LTC4412 -> 6xUSB_PowMet-rescue:LTC4412; Desc (none) -> Testing pass; Description (none) -> LTC4412 - Low Loss PowerPath Controller in ThinSOT; Manufacturer (none) -> Linear Technology; Part Number (none) -> LTC4412ES6#TRMPBF
- U13: symbol LM3150 -> 6xUSB_PowMet-rescue:LM3150; Description (none) -> DC/DC Cntrlr Single-OUT Step Down 1000kHz 14-Pin HTSSOP EP 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; Manufacturer (none) -> Texas Instruments; Part Number (none) -> LM3150MH/NOPB
- U9: symbol FE1.1s -> 6xUSB_PowMet-rescue:FE1.1s; Description (none) -> USB 2.0 HIGH SPEED 4-PORT HUB CONTROLLER; Manufacturer (none) -> Terminus; Part Number (none) -> FE1.1s-BSOP28B
- Y1: footprint Crystals:Crystal_SMD_5032_4Pads -> Crystals:Crystal_HC49-SD_SMD; symbol CRYSTAL_SMD -> Device:Crystal_Small; Description (none) -> Crystal 12MHz ±30ppm (Tol) ±30ppm (Stability) 18pF FUND 40O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; Manufacturer (none) -> TXC Corporation; Part Number (none) -> 9C-12.000MAAJ-T
Connections:
- net labels added: LED1, MC_ST, PB0_40, TESTJ, VDC, VDD, WE-TVS_824001
- net labels removed: +3.3V, 1V8, PC6_25, PC7_26
- wire segments 177 -> 268
- no-connect marks 3 -> 5
Other:
- note added: "4 port USB 2.0 hub"
- note added: "Automatic power switching"
- note added: "Power Supply"
- moved on the sheet: C37, C38, C39, C40, C41, C42, C43, D10, D11, D9, L3, Q1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
